Commit message: SVD commit

File: src/devel_packages/orio/panda_arm_hand.urdf (robot description, URDF)
Before this commit: robot panda, 12 links, 11 joints
Joints:
- joint panda_hand_joint: origin xyz=0 0 -0.04 rpy=0 0 -0.7853981633974483 -> xyz=0 0 0 rpy=0 0 -0.7853981633974483
- joint panda_joint8: origin xyz=0 0 0.107 rpy=0 0 0 -> xyz=0 0 0.17 rpy=0 0 0
